File: pcbs/common/left.kicad_sch (KiCad schematic)
At the start: 96 parts, among them J2 TRS, SW22 SW_Push, SW23 SW_Push

Commit message: schem check, outline done, drc done
Parts:
- removed JP1: SolderJumper_2_Bridged, Jumper:SolderJumper-2_P1.3mm_Open_RoundedPad1.0x1.5mm, symbol Jumper:SolderJumper_2_Bridged
- renumbered EXLED2 to LED16, EXLED1 to LED17
Changed lines of the file:
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@@
 	)
 	(junction
-		(at 261.62 190.5)
-		(diameter 0)
-		(color 0 0 0 0)
-	)
-	(junction
-		(at 208.28 193.04)
-		(diameter 0)
-		(color 0 0 0 0)
-	)
-	(junction
 		(at 231.14 227.33)
 		(diameter 0)
@@
 	)
 	(junction
-		(at 208.28 200.66)
-		(diameter 0)
-		(color 0 0 0 0)
-	)
-	(junction
 		(at 215.9 262.89)
 		(diameter 0)
@@
 	)
 	(no_connect
-		(at 50.8 60.96)
+		(at 193.04 252.73)
 	)
 	(no_connect
-		(at 284.48 234.95)
+		(at 50.8 60.96)
 	)
 	(no_connect
@@
 	(wire
 		(pts
-			(xy 261.62 190.5) (xy 292.1 190.5)
-		)
-		(stroke
-			(width 0)
-			(type default)
-		)
-	)
-	(wire
-		(pts
 			(xy 233.68 34.29) (xy 233.68 36.83)
 		)
@@
 	(wire
 		(pts
-			(xy 182.88 193.04) (xy 182.88 252.73)
-		)
-		(stroke
-			(width 0)
-			(type default)
-		)
-	)
-	(wire
-		(pts
 			(xy 114.3 101.6) (xy 124.46 101.6)
 		)
@@
 	(wire
 		(pts
-			(xy 182.88 193.04) (xy 208.28 193.04)
-		)
-		(stroke
-			(width 0)
-			(type default)
-		)
-	)
-	(wire
-		(pts
 			(xy 111.76 143.51) (xy 120.015 143.51)
 		)
@@
 	(wire
 		(pts
-			(xy 208.28 193.04) (xy 284.48 193.04)
-		)
-		(stroke
-			(width 0)
-			(type default)
-		)
-	)
-	(wire
-		(pts
 			(xy 91.44 114.3) (xy 91.44 120.65)
 		)
@@
 	(wire
 		(pts
-			(xy 284.48 215.9) (xy 284.48 219.71)
-		)
-		(stroke
-			(width 0)
-			(type default)
-		)
-	)
-	(wire
-		(pts
 			(xy 269.24 234.95) (xy 269.24 237.49)
 		)
@@
 	(wire
 		(pts
-			(xy 292.1 190.5) (xy 292.1 227.33)
-		)
-		(stroke
-			(width 0)
-			(type default)
-		)
-	)
-	(wire
-		(pts
 			(xy 73.66 100.33) (xy 81.28 100.33)
 		)
@@
 	(wire
 		(pts
-			(xy 143.51 101.6) (xy 152.4 101.6)
+			(xy 269.24 270.51) (xy 285.75 270.51)
 		)
 		(stroke
@@
 	(wire
 		(pts
-			(xy 193.04 234.95) (xy 193.04 237.49)
+			(xy 143.51 101.6) (xy 152.4 101.6)
 		)
 		(stroke
@@
 	(wire
 		(pts
-			(xy 284.48 193.04) (xy 284.48 200.66)
+			(xy 193.04 234.95) (xy 193.04 237.49)
 		)
 		(stroke
@@
 	(wire
 		(pts
-			(xy 193.04 252.73) (xy 182.88 252.73)
-		)
-		(stroke
-			(width 0)
-			(type default)
-		)
-	)
-	(wire
-		(pts
 			(xy 48.26 176.53) (xy 48.26 173.99)
 		)
@@
 	)
 	(label "LED"
-		(at 269.24 270.51 270)
+		(at 284.48 270.51 0)
 		(fields_autoplaced yes)
 		(effects
@@
 				(size 1.27 1.27)
 			)
-			(justify right bottom)
+			(justify left bottom)
 		)
 	)
@@
 				)
 				(path "/4cc5d416-57f5-4147-8183-e03ae6b1198a/089db7cd-2934-428b-a62a-55e0735649ba"
-					(reference "LED17")
+					(reference "LED19")
 					(unit 1)
 				)
@@
 				)
 				(path "/4cc5d416-57f5-4147-8183-e03ae6b1198a/089db7cd-2934-428b-a62a-55e0735649ba"
-					(reference "LED18")
+					(reference "LED20")
 					(unit 1)
 				)
@@
 				)
 				(path "/4cc5d416-57f5-4147-8183-e03ae6b1198a/089db7cd-2934-428b-a62a-55e0735649ba"
-					(reference "LED21")
+					(reference "LED23")
 					(unit 1)
 				)
@@
 				)
 				(path "/4cc5d416-57f5-4147-8183-e03ae6b1198a/089db7cd-2934-428b-a62a-55e0735649ba"
-					(reference "LED19")
+					(reference "LED21")
 					(unit 1)
 				)
@@
 	)
 	(symbol
-		(lib_id "Jumper:SolderJumper_2_Bridged")
-		(at 208.28 196.85 90)
-		(unit 1)
-		(exclude_from_sim no)
-		(in_bom yes)
-		(on_board yes)
-		(dnp no)
-		(fields_autoplaced yes)
-		(property "Reference" "JP1"
-			(at 210.82 195.58 90)
-			(effects
-				(font
-					(size 1.27 1.27)
-				)
-				(justify right)
-			)
-		)
-		(property "Value" "SolderJumper_2_Bridged"
-			(at 210.82 198.12 90)
-			(effects
-				(font
-					(size 1.27 1.27)
-				)
-				(justify right)
-			)
-		)
-		(property "Footprint" "Jumper:SolderJumper-2_P1.3mm_Open_RoundedPad1.0x1.5mm"
-			(at 208.28 196.85 0)
-			(effects
-				(font
-					(size 1.27 1.27)
-				)
-				(hide yes)
-			)
-		)
-		(property "Datasheet" "~"
-			(at 208.28 196.85 0)
-			(effects
-				(font
-					(size 1.27 1.27)
-				)
-				(hide yes)
-			)
-		)
-		(property "Description" ""
-			(at 208.28 196.85 0)
-			(effects
-				(font
-					(size 1.27 1.27)
-				)
-				(hide yes)
-			)
-		)
-		(pin "1"
-		)
-		(pin "2"
-		)
-		(instances
-			(project "Gecko_choc"
-				(path "/4cc5d416-57f5-4147-8183-e03ae6b1198a/089db7cd-2934-428b-a62a-55e0735649ba"
-					(reference "JP1")
-					(unit 1)
-				)
-			)
-		)
-	)
-	(symbol
 		(lib_id "Device:C_Small")
 		(at 124.46 104.14 0)
@@
 		(on_board yes)
 		(dnp no)
-		(property "Reference" "EXLED1"
+		(property "Reference" "LED17"
 			(at 213.995 268.605 0)
 			(effects
@@
 			(project "Gecko_choc"
 				(path "/4cc5d416-57f5-4147-8183-e03ae6b1198a/089db7cd-2934-428b-a62a-55e0735649ba"
-					(reference "EXLED1")
+					(reference "LED17")
 					(unit 1)
 				)
@@
 		(on_board yes)
 		(dnp no)
-		(property "Reference" "EXLED2"
+		(property "Reference" "LED16"
 			(at 217.805 257.175 0)
 			(effects
@@
 			(project "Gecko_choc"
 				(path "/4cc5d416-57f5-4147-8183-e03ae6b1198a/089db7cd-2934-428b-a62a-55e0735649ba"
-					(reference "EXLED2")
+					(reference "LED16")
 					(unit 1)
 				)
@@
 				)
 				(path "/4cc5d416-57f5-4147-8183-e03ae6b1198a/089db7cd-2934-428b-a62a-55e0735649ba"
-					(reference "LED16")
+					(reference "LED18")
 					(unit 1)
 				)
@@
 				)
 				(path "/4cc5d416-57f5-4147-8183-e03ae6b1198a/089db7cd-2934-428b-a62a-55e0735649ba"
-					(reference "LED20")
+					(reference "LED22")
 					(unit 1)
 				)
@@
 		(on_board yes)
 		(dnp no)
-		(fields_autoplaced yes)
 		(property "Reference" "J2"
 			(at 270.51 28.575 0)

Commit message: renumber switches, git status
Parts:
- renumbered SW23 to SW16, SW22 to SW17
Changed lines of the file:
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@@
 				)
 				(path "/4cc5d416-57f5-4147-8183-e03ae6b1198a/089db7cd-2934-428b-a62a-55e0735649ba"
-					(reference "SW21")
+					(reference "SW23")
 					(unit 1)
 				)
@@
 		(on_board yes)
 		(dnp no)
-		(property "Reference" "SW22"
+		(property "Reference" "SW17"
 			(at 200.66 147.574 0)
 			(effects
@@
 			(project "Gecko_choc"
 				(path "/4cc5d416-57f5-4147-8183-e03ae6b1198a/089db7cd-2934-428b-a62a-55e0735649ba"
-					(reference "SW22")
+					(reference "SW17")
 					(unit 1)
 				)
@@
 				)
 				(path "/4cc5d416-57f5-4147-8183-e03ae6b1198a/089db7cd-2934-428b-a62a-55e0735649ba"
-					(reference "SW19")
+					(reference "SW21")
 					(unit 1)
 				)
@@
 		(on_board yes)
 		(dnp no)
-		(property "Reference" "SW23"
+		(property "Reference" "SW16"
 			(at 214.63 147.574 0)
 			(effects
@@
 			(project "Gecko_choc"
 				(path "/4cc5d416-57f5-4147-8183-e03ae6b1198a/089db7cd-2934-428b-a62a-55e0735649ba"
-					(reference "SW23")
+					(reference "SW16")
 					(unit 1)
 				)
@@
 				)
 				(path "/4cc5d416-57f5-4147-8183-e03ae6b1198a/089db7cd-2934-428b-a62a-55e0735649ba"
-					(reference "SW17")
+					(reference "SW19")
 					(unit 1)
 				)
@@
 				)
 				(path "/4cc5d416-57f5-4147-8183-e03ae6b1198a/089db7cd-2934-428b-a62a-55e0735649ba"
-					(reference "SW16")
+					(reference "SW18")
 					(unit 1)
 				)
@@
 				)
 				(path "/4cc5d416-57f5-4147-8183-e03ae6b1198a/089db7cd-2934-428b-a62a-55e0735649ba"
-					(reference "SW18")
+					(reference "SW20")
 					(unit 1)
 				)
@@
 				)
 				(path "/4cc5d416-57f5-4147-8183-e03ae6b1198a/089db7cd-2934-428b-a62a-55e0735649ba"
-					(reference "SW20")
+					(reference "SW22")
 					(unit 1)
 				)
