File: pcbs/common/right.kicad_sch (KiCad schematic)
At the start: 96 parts, among them J2 TRS

Commit message: schem check, outline done, drc done
Parts:
- removed rJP1: SolderJumper_2_Bridged, Jumper:SolderJumper-2_P1.3mm_Open_RoundedPad1.0x1.5mm, symbol Jumper:SolderJumper_2_Bridged
Changed lines of the file:
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@@
 	)
 	(junction
-		(at 203.2 200.66)
-		(diameter 0)
-		(color 0 0 0 0)
-	)
-	(junction
 		(at 241.3 208.28)
 		(diameter 0)
@@
 	)
 	(no_connect
-		(at 279.4 234.95)
+		(at 187.96 252.73)
 	)
 	(no_connect
@@
 	(wire
 		(pts
-			(xy 177.8 193.04) (xy 203.2 193.04)
-		)
-		(stroke
-			(width 0)
-			(type default)
-		)
-	)
-	(wire
-		(pts
 			(xy 114.3 33.02) (xy 120.65 33.02)
 		)
@@
 	(wire
 		(pts
-			(xy 177.8 193.04) (xy 177.8 252.73)
-		)
-		(stroke
-			(width 0)
-			(type default)
-		)
-	)
-	(wire
-		(pts
 			(xy 218.44 219.71) (xy 218.44 215.9)
 		)
@@
 	(wire
 		(pts
+			(xy 278.13 270.51) (xy 264.16 270.51)
+		)
+		(stroke
+			(width 0)
+			(type default)
+		)
+	)
+	(wire
+		(pts
 			(xy 248.92 200.66) (xy 264.16 200.66)
 		)
@@
 	(wire
 		(pts
-			(xy 187.96 252.73) (xy 177.8 252.73)
-		)
-		(stroke
-			(width 0)
-			(type default)
-		)
-	)
-	(wire
-		(pts
 			(xy 264.16 252.73) (xy 264.16 255.27)
 		)
@@
 	)
 	(label "LED"
-		(at 264.16 270.51 270)
+		(at 278.13 270.51 0)
 		(fields_autoplaced yes)
 		(effects
@@
 				(size 1.27 1.27)
 			)
-			(justify right bottom)
+			(justify left bottom)
 		)
 	)
@@
 					(unit 1)
 				)
-			)
-		)
-	)
-	(symbol
-		(lib_id "Jumper:SolderJumper_2_Bridged")
-		(at 203.2 196.85 90)
-		(unit 1)
-		(exclude_from_sim no)
-		(in_bom yes)
-		(on_board yes)
-		(dnp no)
-		(fields_autoplaced yes)
-		(property "Reference" "rJP1"
-			(at 205.74 195.58 90)
-			(effects
-				(font
-					(size 1.27 1.27)
-				)
-				(justify right)
-			)
-		)
-		(property "Value" "SolderJumper_2_Bridged"
-			(at 205.74 198.12 90)
-			(effects
-				(font
-					(size 1.27 1.27)
-				)
-				(justify right)
-			)
-		)
-		(property "Footprint" "Jumper:SolderJumper-2_P1.3mm_Open_RoundedPad1.0x1.5mm"
-			(at 203.2 196.85 0)
-			(effects
-				(font
-					(size 1.27 1.27)
-				)
-				(hide yes)
-			)
-		)
-		(property "Datasheet" "~"
-			(at 203.2 196.85 0)
-			(effects
-				(font
-					(size 1.27 1.27)
-				)
-				(hide yes)
-			)
-		)
-		(property "Description" ""
-			(at 203.2 196.85 0)
-			(effects
-				(font
-					(size 1.27 1.27)
-				)
-				(hide yes)
-			)
-		)
-		(pin "1"
-		)
-		(pin "2"
-		)
-		(instances
-			(project "right"
-				(path "/04ecfb8d-8dc8-41d9-b176-68a9b73f1e5e"
-					(reference "rJP1")
-					(unit 1)
-				)
-			)
-			(project "Gecko_choc"
-				(path "/4cc5d416-57f5-4147-8183-e03ae6b1198a/50d96a5e-3d25-4129-9495-15388c76587f"
-					(reference "rJP1")
-					(unit 1)
-				)

Commit message: renumber switches, git status
Parts:
- renumbered rSW23 to rSW16, rSW22 to rSW17
Changed lines of the file:
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@@
 				)
 				(path "/4cc5d416-57f5-4147-8183-e03ae6b1198a/50d96a5e-3d25-4129-9495-15388c76587f"
-					(reference "rSW16")
+					(reference "rSW18")
 					(unit 1)
 				)
@@
 				)
 				(path "/4cc5d416-57f5-4147-8183-e03ae6b1198a/50d96a5e-3d25-4129-9495-15388c76587f"
-					(reference "rSW17")
+					(reference "rSW19")
 					(unit 1)
 				)
@@
 				)
 				(path "/4cc5d416-57f5-4147-8183-e03ae6b1198a/50d96a5e-3d25-4129-9495-15388c76587f"
-					(reference "rSW21")
+					(reference "rSW23")
 					(unit 1)
 				)
@@
 		(on_board yes)
 		(dnp no)
-		(property "Reference" "rSW22"
+		(property "Reference" "rSW17"
 			(at 194.31 147.574 0)
 			(effects
@@
 			(project "Gecko_choc"
 				(path "/4cc5d416-57f5-4147-8183-e03ae6b1198a/50d96a5e-3d25-4129-9495-15388c76587f"
-					(reference "rSW22")
+					(reference "rSW17")
 					(unit 1)
 				)
@@
 					(size 1 1)
 				)
+				(hide yes)
 			)
 		)
@@
 				)
 				(path "/4cc5d416-57f5-4147-8183-e03ae6b1198a/50d96a5e-3d25-4129-9495-15388c76587f"
-					(reference "rSW19")
+					(reference "rSW21")
 					(unit 1)
 				)
@@
 				)
 				(path "/4cc5d416-57f5-4147-8183-e03ae6b1198a/50d96a5e-3d25-4129-9495-15388c76587f"
-					(reference "rSW20")
+					(reference "rSW22")
 					(unit 1)
 				)
@@
 				)
 				(path "/4cc5d416-57f5-4147-8183-e03ae6b1198a/50d96a5e-3d25-4129-9495-15388c76587f"
-					(reference "rSW18")
+					(reference "rSW20")
 					(unit 1)
 				)
@@
 		(on_board yes)
 		(dnp no)
-		(property "Reference" "rSW23"
+		(property "Reference" "rSW16"
 			(at 209.55 147.574 0)
 			(effects
@@
 			(project "Gecko_choc"
 				(path "/4cc5d416-57f5-4147-8183-e03ae6b1198a/50d96a5e-3d25-4129-9495-15388c76587f"
-					(reference "rSW23")
+					(reference "rSW16")
 					(unit 1)
 				)
